File: pcb/sat_control_shield/kicad/BSAT - Control Shield.kicad_pcb (KiCad board)
At the start: 2 copper layers, 77 x 77 mm, 19 parts, among them P1 POWER, U1 ARDUINO_NANO_V3.0, U2 74HC4052E

Commit message: feat(control-shield): Sensor de temperatura HTU21D añadido.
Parts:
- added S7: HTU21D-MODULE, boscoverysat:HTU21D-MODULE, F.Cu at (166.0, 113.0)
Routing:
- net /SCL: track 180.8 -> 204.8 mm
- net /SDA: track 147.7 -> 142.3 mm
Changed lines of the file:
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@@
 (kicad_pcb (version 4) (host pcbnew 4.0.2+e4-6225~38~ubuntu14.04.1-stable)
   (general
-    (links 44)
+    (links 48)
     (no_connects 0)
     (area 110.424999 44.924999 187.575001 122.075001)
     (thickness 1.6)
     (drawings 35)
-    (tracks 182)
+    (tracks 189)
     (zones 0)
-    (modules 19)
+    (modules 20)
     (nets 45)
   )
@@
     (pad 1 thru_hole circle (at 0 0) (size 2.5 2.5) (drill 0.5) (layers B.Cu)
       (net 2 GNDREF))
+  )
+  (module boscoverysat:HTU21D-MODULE (layer F.Cu)
+    (at 166 113 90)
+    (fp_text reference S7 (at 3.81 -6.096 90) (layer F.SilkS)
+      (effects (font (size 1 1) (thickness 0.15)))
+    )
+    (fp_text value HTU21D-MODULE (at 3.81 -8.128 90) (layer F.SilkS)
+      (effects (font (size 1 1) (thickness 0.15)))
+    )
+    (fp_circle (center 8.382 -11.43) (end 8.382 -13.462) (layer F.SilkS) (width 0.15))
+    (fp_circle (center -0.762 -11.43) (end -0.762 -13.462) (layer F.SilkS) (width 0.15))
+    (fp_line (start -3.81 0.762) (end -3.81 -14.478) (layer F.SilkS) (width 0.15))
+    (fp_line (start -3.81 -14.478) (end 11.43 -14.478) (layer F.SilkS) (width 0.15))
+    (fp_line (start 11.43 -14.478) (end 11.43 0.762) (layer F.SilkS) (width 0.15))
+    (fp_line (start 11.43 0.762) (end -3.81 0.762) (layer F.SilkS) (width 0.15))
+    (fp_text user SCL (at 7.62 -3.556 180) (layer F.SilkS)
+      (effects (font (size 0.75 0.75) (thickness 0.15)))
+    )
+    (fp_text user SDA (at 5.08 -3.556 180) (layer F.SilkS)
+      (effects (font (size 0.75 0.75) (thickness 0.15)))
+    )
+    (fp_text user GND (at 2.54 -3.556 180) (layer F.SilkS)
+      (effects (font (size 0.75 0.75) (thickness 0.15)))
+    )
+    (fp_text user VCC (at 0 -3.556 180) (layer F.SilkS)
+      (effects (font (size 0.75 0.75) (thickness 0.15)))
+    )
+    (pad 1 thru_hole oval (at 0 0 90) (size 2.25 4) (drill 0.5) (layers B.Cu B.Mask)
+      (net 6 +3V3))
+    (pad 2 thru_hole oval (at 2.54 0 90) (size 2.25 4) (drill 0.5) (layers B.Cu B.Mask)
+      (net 2 GNDREF))
+    (pad 3 thru_hole oval (at 5.08 0 90) (size 2.25 4) (drill 0.5) (layers B.Cu B.Mask)
+      (net 4 /SDA))
+    (pad 4 thru_hole oval (at 7.62 0 90) (size 2.25 4) (drill 0.5) (layers B.Cu B.Mask)
+      (net 5 /SCL))
   )
   (gr_text V1.1 (at 163.5 99.5) (layer B.Cu)
@@
   (segment (start 112 104.5) (end 112.04 104.54) (width 0.75) (layer B.Cu) (net 2))
   (segment (start 112.04 104.54) (end 112 104.54) (width 0.75) (layer B.Cu) (net 2))
-  (segment (start 145 97.72) (end 148.72 97.72) (width 0.5) (layer B.Cu) (net 4))
-  (segment (start 174.54 107.96) (end 174.54 105) (width 0.5) (layer B.Cu) (net 4))
-  (segment (start 173 109.5) (end 174.54 107.96) (width 0.5) (layer B.Cu) (net 4))
-  (segment (start 151.5 109.5) (end 173 109.5) (width 0.5) (layer B.Cu) (net 4))
-  (segment (start 150 108) (end 151.5 109.5) (width 0.5) (layer B.Cu) (net 4))
-  (segment (start 150 99) (end 150 108) (width 0.5) (layer B.Cu) (net 4))
-  (segment (start 148.72 97.72) (end 150 99) (width 0.5) (layer B.Cu) (net 4))
+  (segment (start 174.54 105) (end 174.54 106.96) (width 0.5) (layer B.Cu) (net 4) (status C00000))
+  (segment (start 174.54 106.96) (end 173.58 107.92) (width 0.5) (layer B.Cu) (net 4) (status 400000))
+  (segment (start 173.58 107.92) (end 166 107.92) (width 0.5) (layer B.Cu) (net 4) (status 800000))
+  (segment (start 145 97.72) (end 147.72 97.72) (width 0.5) (layer B.Cu) (net 4) (status 400000))
+  (segment (start 154.92 107.92) (end 166 107.92) (width 0.5) (layer B.Cu) (net 4) (status 800000))
+  (segment (start 149.5 102.5) (end 154.92 107.92) (width 0.5) (layer B.Cu) (net 4))
+  (segment (start 149.5 99.5) (end 149.5 102.5) (width 0.5) (layer B.Cu) (net 4))
+  (segment (start 147.72 97.72) (end 149.5 99.5) (width 0.5) (layer B.Cu) (net 4))
   (segment (start 129 65.92) (end 127.58 65.92) (width 0.5) (layer B.Cu) (net 4))
   (segment (start 127.58 65.92) (end 126.5 67) (width 0.5) (layer B.Cu) (net 4))
@@
   (segment (start 166.38 65.12) (end 172 65.12) (width 0.5) (layer B.Cu) (net 4))
   (segment (start 172 65.12) (end 174.62 65.12) (width 0.5) (layer B.Cu) (net 4))
+  (segment (start 174.62 65.12) (end 176 66.5) (width 0.5) (layer B.Cu) (net 4))
+  (segment (start 176 66.5) (end 176 100.5) (width 0.5) (layer B.Cu) (net 4))
+  (segment (start 176 100.5) (end 174.54 101.96) (width 0.5) (layer B.Cu) (net 4))
   (segment (start 174.54 101.96) (end 174.54 105) (width 0.5) (layer B.Cu) (net 4))
-  (segment (start 176 100.5) (end 174.54 101.96) (width 0.5) (layer B.Cu) (net 4))
-  (segment (start 176 66.5) (end 176 100.5) (width 0.5) (layer B.Cu) (net 4))
-  (segment (start 174.62 65.12) (end 176 66.5) (width 0.5) (layer B.Cu) (net 4))
   (segment (start 145 97.72) (end 146.78 97.72) (width 0.5) (layer B.Cu) (net 4))
+  (segment (start 166 105.38) (end 153.88 105.38) (width 0.5) (layer B.Cu) (net 5) (status 400000))
+  (segment (start 150.5 95.86) (end 149.82 95.18) (width 0.5) (layer B.Cu) (net 5))
+  (segment (start 150.5 102) (end 150.5 95.86) (width 0.5) (layer B.Cu) (net 5))
+  (segment (start 153.88 105.38) (end 150.5 102) (width 0.5) (layer B.Cu) (net 5))
   (segment (start 142 65.46) (end 148.5 65.46) (width 0.5) (layer B.Cu) (net 5))
   (segment (start 148.5 65.46) (end 155 65.46) (width 0.5) (layer B.Cu) (net 5))
@@
   (segment (start 149.82 95.18) (end 153.5 91.5) (width 0.5) (layer B.Cu) (net 5))
   (segment (start 146.82 95) (end 146.5 94.68) (width 0.5) (layer B.Cu) (net 5))
+  (segment (start 145 112.96) (end 165.96 112.96) (width 1) (layer B.Cu) (net 6) (status C00000))
+  (segment (start 165.96 112.96) (end 166 113) (width 1) (layer B.Cu) (net 6) (status C00000))
+  (segment (start 166 113) (end 177.5 113) (width 1) (layer B.Cu) (net 6) (status 400000))
+  (segment (start 177.5 113) (end 182.16 108.34) (width 1) (layer B.Cu) (net 6))
+  (segment (start 182.16 108.34) (end 182.16 105) (width 1) (layer B.Cu) (net 6) (status 800000))
   (segment (start 142 57.84) (end 148.5 57.84) (width 1) (layer B.Cu) (net 6))
   (segment (start 148.5 57.84) (end 155 57.84) (width 1) (layer B.Cu) (net 6))
@@
   (segment (start 161.5 57.84) (end 161.84 57.5) (width 1) (layer B.Cu) (net 6))
   (segment (start 161.84 57.5) (end 172 57.5) (width 1) (layer B.Cu) (net 6))
-  (segment (start 145 112.96) (end 177.54 112.96) (width 1) (layer B.Cu) (net 6))
-  (segment (start 177.54 112.96) (end 182.16 108.34) (width 1) (layer B.Cu) (net 6))
-  (segment (start 182.16 108.34) (end 182.16 105) (width 1) (layer B.Cu) (net 6))
   (segment (start 182.16 105) (end 182.16 61.66) (width 1) (layer B.Cu) (net 6))
   (segment (start 182.16 61.66) (end 178 57.5) (width 1) (layer B.Cu) (net 6))
